File: KiCAD/new_ledMatrix/new_ledMatrix.kicad_pcb (KiCad board)
At the start: 2 copper layers, 72.6 x 39.1 mm, 62 parts

Commit message: via holes moved
Parts:
- moved TP4 2.36 mm to (126.4, 95.0)
Routing:
- net +5V: track 504.8 -> 349.0 mm, vias 59 -> 55
- net Net-(D56-DOUT): track 4.10 -> 7.18 mm
- net GND: track 23.4 -> 26.0 mm
- net Net-(D16-DOUT): track 10.3 -> 9.37 mm
- net Net-(D50-DOUT): track 16.2 -> 15.5 mm
- net Net-(D6-DOUT): track 18.7 -> 18.2 mm
