File: KiCAD/new_ledMatrix/new_ledMatrix.kicad_sch (KiCad schematic)
At the start: 74 parts

Commit message: upadted pcb to ver7
Parts:
- removed C1: 1000uF, Capacitor_SMD:CP_Elec_10x10.5, symbol Device:C_Polarized_Small
- added c11, c12, c13, c14, c16, c17, c18, c2, c20, c21, c22, c23, c25, c26, c27, c29, c3, c30, c31, c32, c33, c35, c36, c37, c38, c4, c40, c41, c42, c44, c45, c46, c47, c49, c50, c51, c52, c54, c55, c56, c6, c7, c8, c9: 0.1uF, Capacitor_SMD:C_0603_1608Metric, symbol Device:C
- renumbered c2 to c1, c4 to c10, c5 to c15, c6 to c19, c7 to c24, c8 to c28, c9 to c34, c10 to c39, c11 to c43, c12 to c48, c3 to c5, c13 to c53
Connections:
- net +5V: now also c28.2, c11.1, c12.1, c13.1, c14.1, c16.2, c17.2, c18.2, c2.1, c20.2, c21.2, c22.2, c23.2, c25.2, c26.2, c27.2, c29.1, c3.1, c30.1, c31.1, c32.1, c33.1, c35.1, c36.1, c37.1, c38.1, c4.1, c40.1, c41.1, c42.1, c44.2, c45.2, c46.2, c47.2, c49.2, c50.2, c51.2, c52.2, c54.2, c55.2, c56.2, c6.1, c7.1, c8.1, c9.1; no longer c28.1
- net GND: now also c28.1, c11.2, c12.2, c13.2, c14.2, c16.1, c17.1, c18.1, c2.2, c20.1, c21.1, c22.1, c23.1, c25.1, c26.1, c27.1, c29.2, c3.2, c30.2, c31.2, c32.2, c33.2, c35.2, c36.2, c37.2, c38.2, c4.2, c40.2, c41.2, c42.2, c44.1, c45.1, c46.1, c47.1, c49.1, c50.1, c51.1, c52.1, c54.1, c55.1, c56.1, c6.2, c7.2, c8.2, c9.2; no longer c28.2
Other:
- moved on the sheet: D1, D10, D11, D12, D13, D14, D15, D16, D17, D18, D19, D2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

Commit message: added daughter a daughterbaord in /Kicad and create the buck boost converter schematic only
Other:
- title: (none) -> LED_matrix
Changed lines of the file:
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@@
 	(generator_version "9.0")
 	(paper "A2")
+	(title_block
+		(title "LED_matrix")
+	)
 	(junction
 		(at 82.55 85.09)
