File: KiCAD/Clone-new_ledMatrix/new_ledMatrix.kicad_pcb (KiCad board)
At the start: 2 copper layers, 72.6 x 39 mm, 62 parts

Commit message: jst connector added
Parts:
- added JST_SH_SM03B: JST_SH_SM03B-SRSS-TB_1x03-1MP_P1.00mm_Horizontal, Connector_JST:JST_SH_SM03B-SRSS-TB_1x03-1MP_P1.00mm_Horizontal, B.Cu at (199.8, 50.5)
- added c10: 0.1uF, Capacitor_SMD:C_0603_1608Metric, B.Cu at (191.5, 47.0)
- added c11: 0.1uF, Capacitor_SMD:C_0603_1608Metric, B.Cu at (208.7, 52.8)
- added c12: 0.1uF, Capacitor_SMD:C_0603_1608Metric, B.Cu at (237.8, 52.8)
- added c13: 0.1uF, Capacitor_SMD:C_0603_1608Metric, B.Cu at (214.6, 58.5)
- added c2: 0.1uF, Capacitor_SMD:C_0603_1608Metric, B.Cu at (202.9, 29.6)
- added c3: 0.1uF, Capacitor_SMD:C_0603_1608Metric, B.Cu at (226.2, 29.6)
- added c4: 0.1uF, Capacitor_SMD:C_0603_1608Metric, B.Cu at (226.1, 35.6)
- added c5: 0.1uF, Capacitor_SMD:C_0603_1608Metric, B.Cu at (197.0, 35.6)
- added c6: 0.1uF, Capacitor_SMD:C_0603_1608Metric, B.Cu at (203.0, 41.3)
- added c7: 0.1uF, Capacitor_SMD:C_0603_1608Metric, B.Cu at (231.8, 41.3)
- added c8: 0.1uF, Capacitor_SMD:C_0603_1608Metric, B.Cu at (249.0, 47.0)
- added c9: 0.1uF, Capacitor_SMD:C_0603_1608Metric, B.Cu at (220.3, 47.0)
- C1: value 1000uF(10x10.5mm) -> 1000uF
Routing:
- net GND: track 25.1 -> 101.8 mm, vias 1 -> 13
- net +5V: track 133.3 -> 187.2 mm, vias 56 -> 68
- net Net-(R1-Pad1): track 4.10 -> 18.4 mm
Other:
- board text added: "minecraft_compass led_matrix"
- board text removed: "minecraft_compass_led_matrix"
