File: KiCAD/Clone-new_ledMatrix/new_ledMatrix.kicad_sch (KiCad schematic)
At the start: 62 parts

Commit message: jst connector added
Parts:
- added c10, c11, c12, c13, c2, c3, c4, c5, c6, c7, c8, c9: 0.1uF, Capacitor_SMD:C_0603_1608Metric, symbol Device:C
Connections:
- net +5V: now also c10.1, c11.2, c12.2, c13.2, c2.1, c3.1, c4.1, c5.2, c6.2, c7.2, c8.1, c9.1
- net GND: now also c10.2, c11.1, c12.1, c13.1, c2.2, c3.2, c4.2, c5.1, c6.1, c7.1, c8.2, c9.2
Other:
- moved on the sheet: C1, D10, D11, D12, D13, D14, D15, D16, D17, D18, D19, D20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
