File: KiCAD/daughter_board/daughter_board.kicad_sch (KiCad schematic)
At the start: 25 parts, among them IC1 QMC5883L, J1 JST, J3 SM02B-SRSS-TB_LF__SN_, U1 TPS61023DRLR, U2 SN74AHCT1G125DBVR, U3 XIAO-ESP32-C3-SMD, U4 MPU-6050

Commit message: reversed the polatrity of the power plug in the daughter board
Parts:
- C1, C4: MPN (none) -> 0603X106K160NT; SKU (none) -> R144118
- C10: MPN (none) -> CL10A475MA8NQNC; SKU (none) -> R144123
- C2, C3: MPN (none) -> CL10A226MO7JZNC; SKU (none) -> R243185
- C5, C6, C8: SKU (none) -> 1415725
- C7: MPN (none) -> 0603B222K500NT; SKU (none) -> R207408
- C9: MPN (none) -> GRM155R71C224MA12D; SKU (none) -> R144018
- IC1: MPN (none) -> QMC5883L; Manufacturer_Part_Number QMC5883L -> (none)
- J1: MPN (none) -> WT100EL-03-T-00; SKU (none) -> R136189
- J3: MPN (none) -> WT100EW-02-0-T-00; SKU (none) -> R136185
- L1: MPN (none) -> XFL4020-222MEC; SKU (none) -> R113961
- R1: MPN (none) -> RC0603FR-07732KL; SKU (none) -> R197181
- R2, R6: MPN (none) -> CRCW0603100KFKEAC; SKU (none) -> R209018
- R3, R4, R5: SKU (none) -> 573846
- R7: MPN (none) -> CRCW0603100KFKEAC.; SKU (none) -> R209018
- U1: MPN (none) -> TPS61023DRLR; SKU (none) -> R216425
- U2: MPN (none) -> SN74AHCT1G125DBVR; SKU (none) -> R201770
- U4: SKU (none) -> 162123
Connections:
- net +BATT: now also J3.1; no longer J3.2
- net -BATT: now also J3.2; no longer J3.1
